File: pcb/Fake7501.sch (EAGLE design)
At the start: 16 parts, among them IC2 XC9572XLTQG100, IC5 HDR, IC6 65(C)02

Commit message: Updated PCB to fix 7501 footprint errors Added GATE_IN functionality in hdl Added support for 65C02S
Parts:
- removed IC5: HDR, commodore:8502-RP
- removed IC6: 65(C)02, commodore:6502-RP
- added IC1: CSG7501, commodore:7501-RP
- added IC3: XC9572XLTQG100, xilinx_xc95XXXxl:XC9572XLTQG100
- added SJ1: (no value), jumper:SJ
- IC2: value XC9572XLTQG100 -> W65C02SP; device xilinx_xc95XXXxl:XC9572XLTQG100 -> commodore:W65C02SP-R
Connections:
- removed net !NMI: IC2.FB3MC2, IC5>NAME.!NMI, IC6A.!NMI
- removed net !RDY': IC2.FB1MC15, IC6A.!RDY
- new net GATE_IN: IC1A.GATE_IN, IC3.FB4MC7
- new net N$1: IC2A.!VP, SJ1.2
- net !IRQ: now also IC1A.!IRQ, IC2A.!IRQ, IC3.FB1MC15; no longer IC2.FB1MC17, IC5>NAME.!IRQ, IC6A.!IRQ
- net !RDY: now also IC1A.!RDY, IC2A.!RDY, IC3.FB1MC10; no longer IC2.FB1MC10, IC5>NAME.!RDY
- net !RESET: now also IC1A.!RESET, IC2A.!RESET, IC3.FB2MC9-I/O/GSR; no longer IC2.FB2MC9-I/O/GSR, IC5>NAME.!RESET, IC6A.!RESET
- net +3V3: now also IC3.VCCINT3,3V@1, IC3.VCCINT3,3V@2, IC3.VCCINT3,3V@3, IC3.VCCIO2,5V/3,3V@1, IC3.VCCIO2,5V/3,3V@2, IC3.VCCIO2,5V/3,3V@3, IC3.VCCIO2,5V/3,3V@4; no longer IC2.VCCINT3,3V@1, IC2.VCCINT3,3V@2, IC2.VCCINT3,3V@3, IC2.VCCIO2,5V/3,3V@1, IC2.VCCIO2,5V/3,3V@2, IC2.VCCIO2,5V/3,3V@3, IC2.VCCIO2,5V/3,3V@4
- net A'0: now also IC2A.A0, IC3.FB1MC9-I/O/GCK1; no longer IC2.FB1MC4, IC6A.A0
- net A'1: now also IC2A.A1, IC3.FB1MC3; no longer IC2.FB1MC8, IC6A.A1
- net A'10: now also IC2A.A10, IC3.FB3MC15; no longer IC2.FB3MC15, IC6A.A10
- net A'11: now also IC2A.A11, IC3.FB3MC18; no longer IC2.FB3MC18, IC6A.A11
- net A'12: now also IC2A.A12, IC3.FB4MC4; no longer IC2.FB4MC3, IC6A.A12
- net A'13: now also IC2A.A13, IC3.FB4MC6; no longer IC2.FB4MC11, IC6A.A13
- net A'14: now also IC2A.A14, IC3.FB4MC14; no longer IC2.FB4MC7, IC6A.A14
- net A'15: now also IC2A.A15, IC3.FB4MC10; no longer IC2.FB4MC18, IC6A.A15
- net A'2: now also IC2A.A2, IC3.FB1MC1; no longer IC2.FB1MC6, IC6A.A2
- net A'3: now also IC2A.A3, IC3.FB1MC12; no longer IC2.FB1MC12, IC6A.A3
- net A'4: now also IC2A.A4, IC3.FB1MC13; no longer IC2.FB1MC13, IC6A.A4
- net A'5: now also IC2A.A5, IC3.FB1MC16; no longer IC2.FB1MC16, IC6A.A5
- net A'6: now also IC2A.A6, IC3.FB3MC1; no longer IC2.FB3MC1, IC6A.A6
- net A'7: now also IC2A.A7, IC3.FB3MC3; no longer IC2.FB3MC3, IC6A.A7
- net A'8: now also IC2A.A8, IC3.FB3MC11; no longer IC2.FB3MC11, IC6A.A8
- net A'9: now also IC2A.A9, IC3.FB3MC7; no longer IC2.FB3MC7, IC6A.A9
- net A0: now also IC1A.A0, IC3.FB3MC2; no longer IC2.FB1MC10-I/O/GCK2, IC5>NAME.A0
- net A1: now also IC1A.A1, IC3.FB1MC7; no longer IC2.FB1MC9-I/O/GCK1, IC5>NAME.A1
- net A10: now also IC1A.A10, IC3.FB3MC4; no longer IC2.FB3MC6, IC5>NAME.A10
- net A11: now also IC1A.A11, IC3.FB3MC6; no longer IC2.FB3MC14, IC5>NAME.A11
- net A12: now also IC1A.A12, IC3.FB3MC14; no longer IC2.FB3MC17, IC5>NAME.A12
- net A13: now also IC1A.A13, IC3.FB3MC17; no longer IC2.FB3MC10, IC5>NAME.A13
- net A14: now also IC1A.A14, IC3.FB4MC3; no longer IC2.FB4MC4, IC5>NAME.A14
- net A15: now also IC1A.A15, IC3.FB4MC11; no longer IC2.FB4MC6, IC5>NAME.A15
- net A2: now also IC1A.A2, IC3.FB1MC10-I/O/GCK2; no longer IC2.FB1MC3, IC5>NAME.A2
- net A3: now also IC1A.A3, IC3.FB1MC4; no longer IC2.FB1MC1, IC5>NAME.A3
- net A4: now also IC1A.A4, IC3.FB1MC8; no longer IC2.FB1MC5, IC5>NAME.A4
- net A5: now also IC1A.A5, IC3.FB1MC6; no longer IC2.FB3MC5, IC5>NAME.A5
- net A6: now also IC1A.A6, IC3.FB3MC5; no longer IC2.FB3MC8, IC5>NAME.A6
- net A7: now also IC1A.A7, IC3.FB3MC8; no longer IC2.FB1MC18, IC5>NAME.A7
- net A8: now also IC1A.A8, IC3.FB1MC18; no longer IC2.FB3MC9, IC5>NAME.A8
- net A9: now also IC1A.A9, IC3.FB3MC9; no longer IC2.FB3MC4, IC5>NAME.A9
- net AEC: now also IC1A.AEC, IC3.FB1MC17; no longer IC2.FB1MC7, IC5>NAME.AEC
- net D'0: now also IC2A.D0, IC3.FB2MC13; no longer IC2.FB2MC13, IC6A.D0
- net D'1: now also IC2A.D1, IC3.FB2MC16; no longer IC2.FB2MC16, IC6A.D1
- net D'2: now also IC2A.D2, IC3.FB2MC17; no longer IC2.FB2MC17, IC6A.D2
- net D'3: now also IC2A.D3, IC3.FB1MC5; no longer IC2.FB2MC4, IC6A.D3
- net D'4: now also IC2A.D4, IC3.FB2MC18; no longer IC2.FB2MC3, IC6A.D4
- net D'5: now also IC2A.D5, IC3.FB4MC17; no longer IC2.FB4MC15, IC6A.D5
- net D'6: now also IC2A.D6, IC3.FB2MC1; no longer IC2.FB4MC16, IC6A.D6
- net D'7: now also IC2A.D7, IC3.FB4MC13; no longer IC2.FB4MC12, IC6A.D7
- net D0: now also IC1A.D0, IC3.FB2MC6; no longer IC2.FB2MC6, IC5>NAME.D0
- net D1: now also IC1A.D1, IC3.FB2MC5; no longer IC2.FB2MC5, IC5>NAME.D1
- net D2: now also IC1A.D2, IC3.FB2MC2; no longer IC2.FB2MC2, IC5>NAME.D2
- net D3: now also IC1A.D3, IC3.FB2MC10; no longer IC2.FB2MC10, IC5>NAME.D3
- net D4: now also IC1A.D4, IC3.GTS1; no longer IC2.GTS1, IC5>NAME.D4
- net D5: now also IC1A.D5, IC3.FB2MC12; no longer IC2.FB2MC12, IC5>NAME.D5
- net D6: now also IC1A.D6, IC3.FB2MC14; no longer IC2.FB2MC14, IC5>NAME.D6
- net D7: now also IC1A.D7, IC3.FB2MC15; no longer IC2.FB2MC15, IC5>NAME.D7
- net GND: now also IC1P.GND, IC3.GND@1, IC3.GND@2, IC3.GND@3, IC3.GND@4, IC3.GND@5, IC3.GND@6, IC3.GND@7, IC3.GND@8, SJ1.1; no longer IC2.GND@1, IC2.GND@2, IC2.GND@3, IC2.GND@4, IC2.GND@5, IC2.GND@6, IC2.GND@7, IC2.GND@8, IC5P.GND, IC6P.GND, IC6P.GND@1
- net N$3: now also IC3.TCK; no longer IC2.TCK
- net N$4: now also IC3.TMS; no longer IC2.TMS
- net N$5: now also IC3.TDI; no longer IC2.TDI
- net N$6: now also IC3.TDO; no longer IC2.TDO
- net P0: now also IC1A.P0, IC3.FB1MC2; no longer IC2.FB1MC2, IC5>NAME.P0
- net P1: now also IC1A.P1, IC3.FB2MC4; no longer IC2.FB2MC18, IC5>NAME.P1
- net P2: now also IC1A.P2, IC3.FB2MC3; no longer IC2.FB4MC17, IC5>NAME.P2
- net P3: now also IC1A.P3, IC3.FB4MC15; no longer IC2.FB2MC1, IC5>NAME.P3
- net P4: now also IC1A.P4, IC3.FB4MC16; no longer IC2.FB4MC13, IC5>NAME.P4
- net P5: now also IC1A.P6, IC3.FB4MC12; no longer IC2.FB4MC10, IC5>NAME.P5
- net P6: now also IC1A.P7, IC3.FB4MC18; no longer IC2.FB4MC14, IC5>NAME.P6
- net PHI: now also IC1A.PHI0, IC2A.PHI0, IC3.FB1MC14-I/O/GCK3; no longer IC2.FB1MC14-I/O/GCK3, IC5>NAME.PHI0, IC6A.PHI0
- net R/!W: now also IC1A.R/!W, IC3.FB2MC8; no longer IC2.FB2MC8, IC5>NAME.R/!W
- net R/!W': now also IC2A.R/!W, IC3.FB2MC11-I/O/GTS2; no longer IC2.FB2MC11-I/O/GTS2, IC6A.R/!W
- net VCC: now also IC1P.VCC, IC2A.!NMI, IC2P.VCC; no longer IC5P.VCC, IC6P.VCC
